File: Shematic/Commande_Schematic.kicad_sch (KiCad schematic)
At the start: 0 parts

Commit message: C avant
Parts:
- added Arduin_Nano_BLE_Remote-Control: Arduino_Nano_v2.x, Module:Arduino_Nano, symbol MCU_Module:Arduino_Nano_v2.x
- added Black-Lithium-1000mAh-45C-3S?: Battery_Lipo, symbol Mylib:Battery_Lipo
Connections:
- new net: Arduin_Nano_BLE_Remote-Control.30 (VIN), Black-Lithium-1000mAh-45C-3S?. (-Cell_2)
- new net: Arduin_Nano_BLE_Remote-Control.4 (GND), Black-Lithium-1000mAh-45C-3S?. (-Cell_2)
Other:
- company: (none) -> Elisa Aerospace Bordeaux
- title: (none) -> Remote Control
Changed lines of the file:
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@@
 (kicad_sch (version 20211123) (generator eeschema)
-  (paper "A4")
+  (paper "A5")
+  (title_block
+    (title "Remote Control")
+    (date "2023-01-26")
+    (company "Elisa Aerospace Bordeaux")
+    (comment 3 "Created under arduino nano BLE and paired with a Spider Bot")
+    (comment 4 "Electrical diagram of a remote control")
+  )
+  (wire (pts (xy 124.46 50.8) (xy 96.52 50.8))
+    (stroke (width 0) (type default) (color 0 0 0 0))
+  )
+  (wire (pts (xy 96.52 58.42) (xy 96.52 88.9))
+    (stroke (width 0) (type default) (color 0 0 0 0))
+  )
+  (wire (pts (xy 58.42 25.4) (xy 58.42 31.75))
+    (stroke (width 0) (type default) (color 0 0 0 0))
+  )
+  (wire (pts (xy 96.52 25.4) (xy 58.42 25.4))
+    (stroke (width 0) (type default) (color 0 0 0 0))
+  )
+  (wire (pts (xy 96.52 88.9) (xy 60.96 88.9))
+    (stroke (width 0) (type default) (color 0 0 0 0))
+  )
+  (wire (pts (xy 124.46 58.42) (xy 96.52 58.42))
+    (stroke (width 0) (type default) (color 0 0 0 0))
+  )
+  (wire (pts (xy 60.96 88.9) (xy 60.96 82.55))
+    (stroke (width 0) (type default) (color 0 0 0 0))
+  )
+  (wire (pts (xy 96.52 50.8) (xy 96.52 25.4))
+    (stroke (width 0) (type default) (color 0 0 0 0))
+  )
+  (symbol (lib_id "MCU_Module:Arduino_Nano_v2.x") (at 60.96 57.15 0) (unit 1)
+    (in_bom yes) (on_board yes) (fields_autoplaced)
+    (property "Reference" "Arduin_Nano_BLE_Remote-Control" (id 0) (at 65.5194 82.55 0)
+      (effects (font (size 1.27 1.27)) (justify left))
+    )
+    (property "Value" "Arduino_Nano_v2.x" (id 1) (at 65.5194 85.09 0)
+      (effects (font (size 1.27 1.27)) (justify left))
+    )
+    (property "Footprint" "Module:Arduino_Nano" (id 2) (at 60.96 57.15 0)
+      (effects (font (size 1.27 1.27) italic) hide)
+    )
+    (property "Datasheet" "https://www.arduino.cc/en/uploads/Main/ArduinoNanoManual23.pdf" (id 3) (at 60.96 57.15 0)
+      (effects (font (size 1.27 1.27)) hide)
+    )
+    (pin "1")
+    (pin "10")
+    (pin "11")
+    (pin "12")
+    (pin "13")
+    (pin "14")
+    (pin "15")
+    (pin "16")
+    (pin "17")
+    (pin "18")
+    (pin "19")
+    (pin "2")
+    (pin "20")
+    (pin "21")
+    (pin "22")
+    (pin "23")
+    (pin "24")
+    (pin "25")
+    (pin "26")
+    (pin "27")
+    (pin "28")
+    (pin "29")
+    (pin "3")
+    (pin "30")
+    (pin "4")
+    (pin "5")
+    (pin "6")
+    (pin "7")
+    (pin "8")
+    (pin "9")
+  )
+  (symbol (lib_id "Mylib:Battery_Lipo") (at 142.24 54.61 0) (unit 1)
+    (in_bom yes) (on_board yes)
+    (property "Reference" "Black-Lithium-1000mAh-45C-3S?" (id 0) (at 142.24 63.5 0)
+      (effects (font (size 1 1)))
+    )
+    (property "Value" "Battery_Lipo" (id 1) (at 142.24 44.45 0)
+      (effects (font (size 1.5 1.5)))
+    )
+    (property "Footprint" "" (id 2) (at 139.7 60.96 0)
+      (effects (font (size 1.27 1.27)) hide)
+    )
+    (property "Datasheet" "" (id 3) (at 139.7 60.96 0)
+      (effects (font (size 1.27 1.27)) hide)
+    )
+    (pin "")
+    (pin "")
+    (pin "")
+    (pin "")
+    (pin "")
+  )
   (sheet_instances
     (path "/" (page "1"))
   )
+  (symbol_instances
+    (path "/0df6ba97-1499-4bf7-8b03-bcf827f3be16"
+      (reference "Arduin_Nano_BLE_Remote-Control") (unit 1) (value "Arduino_Nano_v2.x") (footprint "Module:Arduino_Nano")
+    )
+    (path "/867fc648-4fda-4cd9-9789-c6b1f7ff634d"
+      (reference "Black-Lithium-1000mAh-45C-3S?") (unit 1) (value "Battery_Lipo") (footprint "")
+    )
+  )
 )
