File: Shematic/Robot_Schematic.kicad_sch (KiCad schematic)
At the start: 13 parts

Commit message: C avant
Parts:
- added BF12ABec2APro-Tronik: ESC, symbol Mylib:ESC
- added Black-Lithium-1000mAh-45C-3S: Battery_Lipo, symbol Mylib:Battery_Lipo
- Leg_1: renamed from Patte1; value Motor_Servo -> Ankle_Servo
- Leg_1: renamed from Patte1; value Motor_Servo -> Hip_Servo
- Leg_1: renamed from Patte1; value Motor_Servo -> Knee_Servo
- Leg_2: renamed from Patte3; value Motor_Servo -> Knee_Servo
- Leg_2: renamed from Patte3; value Motor_Servo -> Ankle_Servo
- Leg_2: renamed from Patte3; value Motor_Servo -> Hip_Servo
- Leg_3: renamed from Patte4; value Motor_Servo -> Ankle_Servo
- Leg_3: renamed from Patte4; value Motor_Servo -> Knee_Servo
- Leg_3: renamed from Patte4; value Motor_Servo -> Hip_Servo
- Leg_4: renamed from Patte2; value Motor_Servo -> Hip_Servo
- Leg_4: renamed from Patte2; value Motor_Servo -> Knee_Servo
- Leg_4: renamed from Patte2; value Motor_Servo -> Ankle_Servo
Connections:
- net Gnd: now also BF12ABec2APro-Tronik. (Pin_Signal)
- new net: BF12ABec2APro-Tronik. (Pin_Signal), Black-Lithium-1000mAh-45C-3S. (-Cell_2) (x2)
- new net + 5V: BF12ABec2APro-Tronik. (Pin_Signal)
Other:
- company: (none) -> Elisa Aerospace Bordeaux
- title: (none) -> Spider Bot 
- moved on the sheet: Arduin_Nano_BLE_Robot, Leg_1, Leg_2, Leg_3, Leg_4

Commit message: schematic
Connections:
- net at Black-Lithium-1000mAh-45C-3S. (-Cell_2): no longer BF12ABec2APro-Tronik. (Pin_Signal)
- new net: BF12ABec2APro-Tronik. (Pin_Signal), Black-Lithium-1000mAh-45C-3S. (-Cell_2) (x2)
- now unconnected: Black-Lithium-1000mAh-45C-3S. (-Cell_2)

Commit message: final
Connections:
- net at Black-Lithium-1000mAh-45C-3S. (-Cell_2): no longer BF12ABec2APro-Tronik. (Pin_Signal)
- new net: BF12ABec2APro-Tronik. (Pin_Signal), Black-Lithium-1000mAh-45C-3S. (-Cell_2) (x2)
- now unconnected: Black-Lithium-1000mAh-45C-3S. (-Cell_2)
